File: control_board.sch (EAGLE design)
At the start: 12 parts, among them CON1 EH_B10B-EH, M1 ARDUINO-NANO-3.0

Commit message: BOM update
Parts:
- DS2482-100_L: value Left -> DS2482-100
- DS2482-100_R: value Right -> DS2482-100
- R_SNS_L, R_SNS_R: value 120Ω -> 120
Changed lines of the file:
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@@
 <part name="GND4" library="Isaks Bibliotek" library_urn="urn:adsk.eagle:library:11889733" deviceset="GND" device=""/>
 <part name="SUPPLY5" library="Isaks Bibliotek" library_urn="urn:adsk.eagle:library:11889733" deviceset="5V" device=""/>
-<part name="R_SNS_L" library="CASE-RCL" library_urn="urn:adsk.eagle:library:5287922" deviceset="R1206" device="" package3d_urn="urn:adsk.eagle:package:5332308/3" value="120Ω"/>
-<part name="R_SNS_R" library="CASE-RCL" library_urn="urn:adsk.eagle:library:5287922" deviceset="R1206" device="" package3d_urn="urn:adsk.eagle:package:5332308/3" value="120Ω"/>
-<part name="DS2482-100_L" library="Isaks Bibliotek" library_urn="urn:adsk.eagle:library:11889733" deviceset="DS2482-100" device="" package3d_urn="urn:adsk.eagle:package:13374351/1" value="Left"/>
+<part name="R_SNS_L" library="CASE-RCL" library_urn="urn:adsk.eagle:library:5287922" deviceset="R1206" device="" package3d_urn="urn:adsk.eagle:package:5332308/3" value="120"/>
+<part name="R_SNS_R" library="CASE-RCL" library_urn="urn:adsk.eagle:library:5287922" deviceset="R1206" device="" package3d_urn="urn:adsk.eagle:package:5332308/3" value="120"/>
+<part name="DS2482-100_L" library="Isaks Bibliotek" library_urn="urn:adsk.eagle:library:11889733" deviceset="DS2482-100" device="" package3d_urn="urn:adsk.eagle:package:13374351/1" value="DS2482-100"/>
 <part name="SUPPLY7" library="Isaks Bibliotek" library_urn="urn:adsk.eagle:library:11889733" deviceset="5V" device=""/>
 <part name="GND6" library="Isaks Bibliotek" library_urn="urn:adsk.eagle:library:11889733" deviceset="GND" device=""/>
@@
 <part name="SUPPLY8" library="Isaks Bibliotek" library_urn="urn:adsk.eagle:library:11889733" deviceset="5V" device=""/>
 <part name="GND8" library="Isaks Bibliotek" library_urn="urn:adsk.eagle:library:11889733" deviceset="GND" device=""/>
-<part name="DS2482-100_R" library="Isaks Bibliotek" library_urn="urn:adsk.eagle:library:11889733" deviceset="DS2482-100" device="" package3d_urn="urn:adsk.eagle:package:13374351/1" value="Right"/>
+<part name="DS2482-100_R" library="Isaks Bibliotek" library_urn="urn:adsk.eagle:library:11889733" deviceset="DS2482-100" device="" package3d_urn="urn:adsk.eagle:package:13374351/1" value="DS2482-100"/>
 <part name="SUPPLY6" library="Isaks Bibliotek" library_urn="urn:adsk.eagle:library:11889733" deviceset="5V" device=""/>
 <part name="GND5" library="Isaks Bibliotek" library_urn="urn:adsk.eagle:library:11889733" deviceset="GND" device=""/>
